File: PowerRDP.sch (KiCad schematic (older format))
At the start: 40 parts, among them J1 Conn_01x02_Male, J10 FPGA, J11 FAA LED, J12 Switch, J2 Conn_01x02_Male, J3 Conn_01x02_Male, J4 Conn_01x02_Male, J5 Conn_01x02_Male, J6 Conn_01x02_Male, J7 3.3V, J8 5V, J9 12V, Q1 NTR4003NT1G, U1 Recom_RS3, U2 LM2575-3.3BU, U3 LM2575-5.0BU, U4 LM2575-12BU, U5 TS555

Commit message: Update diodes to something I can buy
Parts:
- D1, D2, D3: footprint Diode_SMD:D_0805_2012Metric_Pad1.15x1.40mm_HandSolder -> Diode_SMD:D_SOD-123
Changed lines of the file:
@@
 F 0 "D1" V 6604 1579 50  0000 L CNN
 F 1 "1N5819" V 6695 1579 50  0000 L CNN
-F 2 "Diode_SMD:D_0805_2012Metric_Pad1.15x1.40mm_HandSolder" H 6650 1500 50  0001 C CNN
+F 2 "Diode_SMD:D_SOD-123" H 6650 1500 50  0001 C CNN
 F 3 "~" H 6650 1500 50  0001 C CNN
 	1    6650 1500
@@
 F 0 "D2" V 6604 2929 50  0000 L CNN
 F 1 "1N5819" V 6695 2929 50  0000 L CNN
-F 2 "Diode_SMD:D_0805_2012Metric_Pad1.15x1.40mm_HandSolder" H 6650 2850 50  0001 C CNN
+F 2 "Diode_SMD:D_SOD-123" H 6650 2850 50  0001 C CNN
 F 3 "~" H 6650 2850 50  0001 C CNN
 	1    6650 2850
@@
 F 0 "D3" V 6654 4179 50  0000 L CNN
 F 1 "1N5819" V 6745 4179 50  0000 L CNN
-F 2 "Diode_SMD:D_0805_2012Metric_Pad1.15x1.40mm_HandSolder" H 6700 4100 50  0001 C CNN
+F 2 "Diode_SMD:D_SOD-123" H 6700 4100 50  0001 C CNN
 F 3 "~" H 6700 4100 50  0001 C CNN
 	1    6700 4100
